File: hardware/electronics/robotic_arm/robotic_arm.kicad_sch (KiCad schematic)
At the start: 2 parts, among them J1 Raspberry_Pi_2_3, U1 815

Commit message: .
Parts:
- removed J1: Raspberry_Pi_2_3, symbol Connector:Raspberry_Pi_2_3
- added C1: 1000uF, symbol Device:C_Polarized
- added C4: 100uF, symbol Device:C_Polarized
- added J1, J2, J3, J4, J5, J6: Conn_01x03_Pin, symbol Connector:Conn_01x03_Pin
Connections:
- net at U1.0 (PWM_0): now also J1.1 (Pin_1)
- net at U1.1 (PWM_1): now also J2.1 (Pin_1)
- net at U1.2 (PWM_2): now also J3.1 (Pin_1)
- net at U1.3 (PWM_3): now also J4.1 (Pin_1)
- net at U1.4 (PWM_4): now also J5.1 (Pin_1)
- net at U1.5 (PWM_5): now also J6.1 (Pin_1)
- net at U1.GND_1 (GND): now also J1.2 (Pin_2), J2.2 (Pin_2), J3.2 (Pin_2), J4.2 (Pin_2), J5.2 (Pin_2), J6.2 (Pin_2)
- net at U1.V+_1 (V+): now also J1.3 (Pin_3), J2.3 (Pin_3), J3.3 (Pin_3), J4.3 (Pin_3), J5.3 (Pin_3), J6.3 (Pin_3)
